File: testing.sch (KiCad schematic (older format))
At the start: 1 part

Commit message: added new lib
Parts:
- added IC?: AT42QT1070-SSU, symbol Adafruit_AT42QT1070_Breakout-eagle-import:AT42QT1070-SSU
Changed lines of the file:
@@
 $Descr A4 11693 8268
 encoding utf-8
-Sheet 1 1
+Sheet 1 2
 Title ""
 Date ""
@@
 	1    0    0    -1
 $EndComp
+$Sheet
+S 6450 3350 1100 800
+U 5F7E2D46
+F0 "Sheet5F7E2D45" 50
+F1 "sensor.sch" 50
+$EndSheet
+$Comp
+L Adafruit_AT42QT1070_Breakout-eagle-import:AT42QT1070-SSU IC?
+U 1 1 5F7E3813
+P 4400 4800
+F 0 "IC?" H 4574 3904 59  0000 C CNN
+F 1 "AT42QT1070-SSU" H 4400 4800 50  0001 C CNN
+F 2 "" H 4400 4800 50  0001 C CNN
+F 3 "" H 4400 4800 50  0001 C CNN
+	1    4400 4800
+	1    0    0    -1
+$EndComp
